Commit message: im confident this is now correct.
- hesai_base is +x forward away from the connector
- pandar points +x left (50.4mm above hesai base)

File: urdf/hesai.urdf.xacro (robot description, xacro)
@@ -50,5 +50,5 @@
     <!-- See page 12 of User Manual -->
     <!-- note that the X axis points left. See manual page 11 -->
-    <origin xyz="0.0 0.0 50.4e-3" rpy="0.0 0.0 0.0"/>
+    <origin xyz="0.0 0.0 50.4e-3" rpy="0.0 0.0 ${pi/2}"/>
     <parent link="hesai_base"/>
     <child link="${lidar_frame}" />
